File: Wheelmod_rs485.brd (EAGLE design)
At the start: 42 x 40 mm, 52 parts, among them IC1 SN75176BPSR, SW1 RST_SW, SW2 HWB_SW, U1 ATMEGA8U2AU, U2 SI8441IS1, U3 MC33887-HSOP, U4 NFET-SOIC8, U5 LDO, X1 MINI-USB, X3 ENC, X5 LOGIC_IN, Y1 SMDRESONATOR

Commit message: Testing
Parts:
- moved R5 8.88 mm to (8.60, 23.5), turned to 0 degrees
- moved IC1 1.46 mm to (9.70, 28.9)
- moved F1 1.13 mm to (8.30, 34.6)
- moved C15 1.01 mm to (11.6, 35.1)
- moved X2 0.68 mm to (4.30, 30.5)
Connections:
- net A: no longer R5.1
- net B: no longer R5.2
- net RX: now also R5.2
- net TX: now also R5.1
Routing:
- net B: track 10.7 -> 7.13 mm, vias 0 -> 1
- net A: track 9.86 -> 7.13 mm
- net N$22: track 7.24 -> 4.78 mm
- net DE: track 7.04 -> 8.50 mm
- net TX: track 7.11 -> 8.39 mm
- net RX: track 15.3 -> 16.3 mm
- net VCC: track 91.9 -> 90.9 mm
- net GND: vias 27 -> 28
